File: Hardware/Logitech Unifying 2242.kicad_pcb (KiCad board)
At the start: 2 copper layers, 22 x 42 mm, 19 parts, among them J1 Bus_M.2_Socket_B, J2 USB, U1 TPS613222ADBV

Commit message: Copper cleanup
Parts:
- renumbered J2 to USB1
Other:
- board text added: "5V"
- board text added: "D+"
- board text added: "D-"
- board text added: "GND"
- board text added: "USB port optional, will hang off edge if placed"
Changed lines of the file:
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@@
     (pad_to_mask_clearance 0)
     (aux_axis_origin 127.6 121.2)
-    (grid_origin 127.6 121.2)
     (pcbplotparams
       (layerselection 0x00010fc_ffffffff)
@@
     (property "ki_keywords" "connector")
     (attr smd)
-    (fp_text reference "J2" (at 0 1.8) (layer "F.SilkS") hide
-        (effects (font (size 1 1) (thickness 0.15)))
+    (fp_text reference "USB1" (at -8.1 -5.3) (layer "F.SilkS")
+        (effects (font (size 0.5 0.5) (thickness 0.1) bold))
     )
     (fp_text value "USB" (at 0 9.09) (layer "F.Fab")
-        (effects (font (size 1 1) (thickness 0.15)))
-    )
-    (fp_text user "USB" (at -8.4 -5.6 unlocked) (layer "F.SilkS")
         (effects (font (size 1 1) (thickness 0.15)))
     )
@@
     (effects (font (size 1 1) (thickness 0.2)) (justify mirror))
   )
-  (gr_text "USB 2.0\n500mA MAX CURRENT" (at 129 83.7) (layer "F.SilkS")
+  (gr_text "D-" (at 139.7 109.3 90) (layer "F.SilkS")
+    (effects (font (size 1 1) (thickness 0.15)) (justify left))
+  )
+  (gr_text "D+" (at 137.7 109.3 90) (layer "F.SilkS")
+    (effects (font (size 1 1) (thickness 0.15)) (justify left))
+  )
+  (gr_text "GND" (at 135.2 109.3 90) (layer "F.SilkS")
+    (effects (font (size 1 1) (thickness 0.15)) (justify left))
+  )
+  (gr_text "5V" (at 142.2 109.3 90) (layer "F.SilkS")
+    (effects (font (size 1 1) (thickness 0.15)) (justify left))
+  )
+  (gr_text "USB 2.0\n500mA MAX CURRENT" (at 129 83.8) (layer "F.SilkS")
     (effects (font (size 1 1) (thickness 0.2) bold) (justify left bottom))
+  )
+  (gr_text "USB port optional, will\nhang off edge if placed" (at 150.8 103) (layer "Cmts.User")
+    (effects (font (size 1 1) (thickness 0.15)) (justify left bottom))
   )
   (dimension (type aligned) (layer "Dwgs.User")
@@
   (via (at 146.1 113.5) (size 0.5) (drill 0.3) (layers "F.Cu" "B.Cu") (free) (net 2))
   (segment (start 142.3975 114.4) (end 143.6325 114.4) (width 0.25) (layer "F.Cu") (net 3))
-  (segment (start 131 117.6) (end 130.8 117.8) (width 0.25) (layer "F.Cu") (net 4))
+  (segment (start 131 117.3) (end 130.6 117.3) (width 0.25) (layer "F.Cu") (net 4))
+  (segment (start 139.85 117.6) (end 142.85 117.6) (width 0.25) (layer "F.Cu") (net 4))
+  (segment (start 129.5 117.3) (end 129.125 116.925) (width 0.25) (layer "F.Cu") (net 4))
+  (segment (start 130.8 117.5) (end 131 117.3) (width 0.25) (layer "F.Cu") (net 4))
+  (segment (start 133.2 117.3) (end 131 117.3) (width 0.25) (layer "F.Cu") (net 4))
+  (segment (start 135.35 117.6) (end 133.5 117.6) (width 0.25) (layer "F.Cu") (net 4))
+  (segment (start 130.6 117.3) (end 129.5 117.3) (width 0.25) (layer "F.Cu") (net 4))
   (segment (start 129.125 116.925) (end 129.125 116.3) (width 0.25) (layer "F.Cu") (net 4))
-  (segment (start 129.125 116.925) (end 129.8 117.6) (width 0.25) (layer "F.Cu") (net 4))
-  (segment (start 139.85 117.6) (end 142.85 117.6) (width 0.25) (layer "F.Cu") (net 4))
-  (segment (start 135.35 117.6) (end 133.5 117.6) (width 0.25) (layer "F.Cu") (net 4))
+  (segment (start 130.8 118.2) (end 130.8 117.5) (width 0.25) (layer "F.Cu") (net 4))
   (segment (start 133.5 117.6) (end 133.2 117.3) (width 0.25) (layer "F.Cu") (net 4))
-  (segment (start 129.8 117.6) (end 130.6 117.6) (width 0.25) (layer "F.Cu") (net 4))
-  (segment (start 133.2 117.3) (end 131.3 117.3) (width 0.25) (layer "F.Cu") (net 4))
-  (segment (start 130.6 117.6) (end 130.8 117.8) (width 0.25) (layer "F.Cu") (net 4))
-  (segment (start 131.3 117.3) (end 131 117.6) (width 0.25) (layer "F.Cu") (net 4))
-  (segment (start 131 117.6) (end 130.6 117.6) (width 0.25) (layer "F.Cu") (net 4))
-  (segment (start 130.8 118.2) (end 130.8 117.8) (width 0.25) (layer "F.Cu") (net 4))
+  (segment (start 130.8 117.5) (end 130.6 117.3) (width 0.25) (layer "F.Cu") (net 4))
   (via (at 139.85 117.6) (size 0.5) (drill 0.3) (layers "F.Cu" "B.Cu") (net 4))
   (via (at 135.35 117.6) (size 0.5) (drill 0.3) (layers "F.Cu" "B.Cu") (net 4))
@@
       )
     )
+  )
+  (zone (net 0) (net_name "") (layers "F.Cu" "Edge.Cuts") (hatch edge 0.5)
+    (connect_pads (clearance 0))
+    (min_thickness 0.25) (filled_areas_thickness no)
+    (keepout (tracks allowed) (vias allowed) (pads allowed) (copperpour not_allowed) (footprints allowed))
+    (fill (thermal_gap 0.5) (thermal_bridge_width 0.5))
+    (polygon
+      (pts
+        (xy 136 114.8)
+        (xy 136.8 114.8)
+        (xy 136.8 116.2)
+        (xy 136 116.2)
+      )
+    )
