File: Hardware/Logitech Unifying 2242.kicad_sch (KiCad schematic)
At the start: 19 parts, among them J1 Bus_M.2_Socket_B, J2 USB, U1 TPS613222ADBV

Commit message: Copper cleanup
Parts:
- renumbered J2 to USB1
Changed lines of the file:
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@@
   (symbol (lib_id "Connector_Generic:Conn_01x04") (at 144.78 91.44 180) (unit 1)
     (in_bom yes) (on_board yes) (dnp no) (fields_autoplaced)
-    (property "Reference" "J2" (at 144.78 80.01 0)
+    (property "Reference" "USB1" (at 144.78 81.28 0)
       (effects (font (size 1.27 1.27)))
     )
-    (property "Value" "USB" (at 144.78 82.55 0)
+    (property "Value" "USB" (at 144.78 83.82 0)
       (effects (font (size 1.27 1.27)))
     )
@@
       (project "Logitech Unifying 2242"
         (path "/1bbba678-0bcb-4cc7-a74d-51164c36ba99"
-          (reference "J2") (unit 1)
+          (reference "USB1") (unit 1)
         )
       )
